File: Commitment-5x12.kicad_pcb (KiCad board)
At the start: 2 copper layers, 234.4 x 118.4 mm, 97 parts, among them J1 Conn_01x13, J2 Conn_01x13, J3 Conn_01x03, J4 Conn_01x04, J5 Conn_01x04, SW1 OS102011MS2QN1, SW2 RotaryEncoder

Commit message: Working toward revision 1
Parts:
- removed JP1: SolderJumper_3_Bridged12, Jumper:SolderJumper-3_P1.3mm_Bridged12_RoundedPad1.0x1.5mm
- removed REF**: OSHW-Logo_5.7x6mm_Copper, Symbol:OSHW-Logo_5.7x6mm_Copper
- removed REF**: KiCad-Logo_6mm_Copper, Symbol:KiCad-Logo_6mm_Copper
- added S1: PTS810, lizard_libs:PTS_180_Tactile_Switch, F.Cu at (76.2, 36.8)
- H3, H4, H5, H6, H7, H8: value 36-4892CT-ND -> 36-4882CT-ND
- J1, J2: footprint lizard_libs:PinHeader_1x13_P2.54mm_Vertical -> lizard_libs:PinSocket_1x12_P2.54mm_Vertical
- moved BAT1 96.6 mm to (199.4, 35.6), turned to 180 degrees
- moved G*** 96.5 mm to (199.4, 35.6)
- moved SW1 77.7 mm to (68.6, 34.8)
- moved J1 2.54 mm to (33.0, 44.5)
- moved J2 2.54 mm to (61.0, 29.2)
Connections:
- J1 pad 1: GND -> Net-(D21-K)
- J1 pad 10: COL 8 -> COL 10
- J1 pad 11: COL 10 -> COL 12
- J1 pad 12: COL 12 -> COL 7
- J1 pad 2: Net-(D21-K) -> COL 1
- J1 pad 3: COL 1 -> GND
- J1 pad 5: GND -> ROW 2
- J1 pad 6: ROW 2 -> ROW 4
- J1 pad 7: ROW 4 -> COL 2
- J1 pad 8: COL 2 -> COL 4
- J1 pad 9: COL 4 -> COL 8
- J2 pad 10: unconnected-(J2-Pin_10-Pad10) -> Net-(J2-Pin_10)
- J2 pad 12: Net-(J2-Pin_12) -> /BAT +
- J2 pad 9: Net-(J2-Pin_9) -> unconnected-(J2-Pin_9-Pad9)
Routing:
- net /BAT +: track 476.9 -> 353.9 mm, vias 10 -> 8
- net Net-(BAT1-+): track 8.19 -> 117.2 mm
- net Net-(J2-Pin_10): track 0.00 -> 47.9 mm, vias 0 -> 1
- net GND: track 80.6 -> 100.0 mm, vias 99 -> 100
- net Net-(J2-Pin_12): track 4.94 -> 0.00 mm
- net Net-(J2-Pin_9): track 4.94 -> 0.00 mm
- net ROW 5: track 299.6 -> 297.1 mm
- net ROW 1: track 215.6 -> 213.1 mm
- net COL 5: track 225.8 -> 223.3 mm
- net ROW 3: track 255.0 -> 252.5 mm
- net COL 6: track 160.2 -> 157.6 mm
- net COL 3: track 209.8 -> 207.3 mm
- net COL 9: track 291.4 -> 288.8 mm
- net COL 11: track 349.5 -> 347.0 mm
Other:
- outline, holes or cut-outs redrawn
