File: Commitment-5x12.kicad_sch (KiCad schematic)
At the start: 94 parts, among them J1 Conn_01x13, J2 Conn_01x13, J3 Conn_01x03, J4 Conn_01x04, J5 Conn_01x04, SW1 OS102011MS2QN1, SW2 RotaryEncoder

Commit message: Working toward revision 1
Parts:
- removed JP1: SolderJumper_3_Bridged12, Jumper:SolderJumper-3_P1.3mm_Bridged12_RoundedPad1.0x1.5mm, symbol Jumper:SolderJumper_3_Bridged12
- added S1: PTS810, lizard_libs:PTS_180_Tactile_Switch, symbol lizard_lib:PTS810
- J1, J2: footprint lizard_libs:PinHeader_1x13_P2.54mm_Vertical -> lizard_libs:PinSocket_1x12_P2.54mm_Vertical; symbol Connector_Generic:Conn_01x13 -> Connector_Generic:Conn_01x12
Connections:
- net BAT +: now also J2.12 (Pin_12)
- net COL 1: now also J1.2 (Pin_2); no longer J1.3 (Pin_3)
- net COL 10: now also J1.10 (Pin_10); no longer J1.11 (Pin_11)
- net COL 12: now also J1.11 (Pin_11); no longer J1.12 (Pin_12)
- net COL 2: now also J1.7 (Pin_7); no longer J1.8 (Pin_8)
- net COL 4: now also J1.8 (Pin_8); no longer J1.9 (Pin_9)
- net COL 7: now also J1.12 (Pin_12); no longer J1.13 (Pin_13)
- net COL 8: now also J1.9 (Pin_9); no longer J1.10 (Pin_10)
- net GND: now also J1.3 (Pin_3), S1.3, S1.4; no longer J1.1 (Pin_1), J1.5 (Pin_5)
- net ROW 2: now also J1.5 (Pin_5); no longer J1.6 (Pin_6)
- net ROW 4: now also J1.6 (Pin_6); no longer J1.7 (Pin_7)
- net at J2.10 (Pin_10): now also S1.1, S1.2
- net at D21.1 (K): now also J1.1 (Pin_1); no longer J1.2 (Pin_2)
- no-connect marks 11 -> 10
Other:
- moved on the sheet: J4, J5

Commit message: working toward rev 1
Parts:
- added M1, M2: ~, lizard_libs:MX_2U_Stabilizer_Mount, symbol lizard_lib:MX_Stabilizer
- MX1, MX10, MX11, MX12, MX13, MX14, MX15, MX16, MX17, MX18, MX19, MX2, MX20, MX21, MX22, MX23, MX24, MX26, MX27, MX28, MX29, MX3, MX31, MX32, MX33, MX34, MX36, MX37, MX38, MX39, MX4, MX41, MX42, MX43, MX44, MX45, MX46, MX47, MX48, MX49, MX5, MX50, MX51, MX52, MX53, MX54, MX55, MX56, MX57, MX58, MX59, MX6, MX60, MX7, MX8, MX9: footprint lizard_libs:SW_Cherry_MX_1.00u_PCB -> lizard_libs:hotswap_keyswitch_reflow
- MX25, MX40: footprint lizard_libs:SW_Cherry_MX_2.00u_PCB -> lizard_libs:hotswap_keyswitch_reflow
